Commit message: graph nav works, missing dynamic configuration

File: mir_description/urdf/include/mir_250_v1.urdf.xacro (robot description, xacro)
@@ -90,5 +90,5 @@
       <parent link="${prefix}base_link" />
       <child link="${prefix}virtual_laser_link" />
-      <origin xyz="0.0 0.0 0.2" rpy="0.0 0.0 0" />
+      <origin xyz="0.0 0.0 0.1914" rpy="0.0 0.0 0" />
     </joint>
     <link name="${prefix}virtual_laser_link">
